File: 555_Timer_Clock.kicad_sch (KiCad schematic)
At the start: 16 parts, among them J1 +5V, J2 CLK_Out, SW1 Trigger, SW2 RST, U1 ICM7555xB

Commit message: nan
Other:
- company: GYRONIX TECHNOLOGIES -> GYRONIX Embedded Systems
Changed lines of the file:
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@@
 		(date "2026-03-26")
 		(rev "1")
-		(company "GYRONIX TECHNOLOGIES")
+		(company "GYRONIX Embedded Systems")
 		(comment 1 "Design Engineer: Gyro Madrona")
 	)
